File: PCB design/schematic_v3/_autosave-schematic_v3.kicad_pcb (KiCad board)
At the start: 4 copper layers, 108 parts, among them IC1 LAN9252, J1 Conn_01x04_Pin, J2 connection_moteur, J3 Conn_01x05_Pin, J4 Conn_01x03_Pin, J5 Conn_01x02_Pin, Q1 AO3400A, U1 HX1188NL, U2 SP3485CN, U3 24FC512-I/ST, U4 LMR14030SQDPRTQ1, U5 STM32F446RETx, U7 AP63203WU, Y1 25MHz, Y2 8MHz

Commit message: 03/06
Parts:
- moved J2 0.82 mm to (226.0, 54.0)
- turned R10 to 0 degrees
Routing:
- net Net-(J2-Pin_3): track 2.83 -> 16.8 mm
- net Net-(J2-Pin_4): track 7.31 -> 8.17 mm

Commit message: pcb updated
Parts:
- removed C50, C51, C57: 100n, Capacitor_SMD:C_0603_1608Metric
- removed C52: 270p, Capacitor_SMD:C_0603_1608Metric
- removed C53, C55: 27u, Capacitor_SMD:C_1206_3216Metric
- removed C56: 10u, Capacitor_SMD:C_1206_3216Metric
- removed C58, C59: 22u, Capacitor_SMD:C_1206_3216Metric
- removed L3: 6.8u, Inductor_SMD:L_Bourns-SRN4018
- removed U7: AP63203WU, Package_TO_SOT_SMD:TSOT-23-6
- added C23: 18p, Capacitor_SMD:C_0603_1608Metric, F.Cu at (160.4, 90.1)
- added C24: 100n, Capacitor_SMD:C_0603_1608Metric, F.Cu at (149.4, 106.0)
- added C25: 100n, Capacitor_SMD:C_0603_1608Metric, F.Cu at (159.1, 109.5)
- added C31: 100n, Capacitor_SMD:C_0603_1608Metric, F.Cu at (142.1, 105.9)
- added C32: 20p, Capacitor_SMD:C_0603_1608Metric, F.Cu at (135.9, 105.9)
- added C34: 100n, Capacitor_SMD:C_0603_1608Metric, B.Cu at (176.7, 102.3)
- added C36: 1u, Capacitor_SMD:C_0603_1608Metric, F.Cu at (133.8, 89.5)
- added C37: 4.7u, Capacitor_SMD:C_0603_1608Metric, F.Cu at (147.2, 95.6)
- added C49: 22u, Capacitor_SMD:C_1206_3216Metric, B.Cu at (164.6, 83.0)
- added F1: 2920L150_60MR, footprints:2920L150_60MR, B.Cu at (176.4, 110.1)
- added H1: MountingHole, MountingHole:MountingHole_3.2mm_M3_Pad_Via, F.Cu at (127.5, 80.2)
- added H2: MountingHole, MountingHole:MountingHole_3.2mm_M3_Pad_Via, F.Cu at (186.5, 115.2)
- added H3: MountingHole, MountingHole:MountingHole_3.2mm_M3_Pad_Via, F.Cu at (127.5, 115.2)
- added H4: MountingHole, MountingHole:MountingHole_3.2mm_M3_Pad_Via, F.Cu at (186.5, 80.2)
- added L2: 6.8u, Inductor_SMD:L_Bourns-SRN4018, B.Cu at (167.5, 89.5)
- added U6: AP63203WU, Package_TO_SOT_SMD:TSOT-23-6, B.Cu at (173.9, 88.5)
- C1, C11, C13, C15, C16, C17, C21, C28, C35: value 0.1u -> 100n
- C10: value 47u -> 1n; footprint Capacitor_SMD:CP_Elec_5x5.4 -> Capacitor_SMD:C_0603_1608Metric; moved to F.Cu
- C18: value 47u -> 1u; footprint Capacitor_SMD:CP_Elec_5x5.4 -> Capacitor_SMD:C_0603_1608Metric; moved to F.Cu
- C20: value 1u -> 100n
- C22: value 0.1u -> 18p
- C26: value 18p -> 47u; footprint Capacitor_SMD:C_0603_1608Metric -> Capacitor_SMD:CP_Elec_5x5.4; moved to B.Cu
- C27: value 18p -> 100n
- C30: value 0.1u -> 100n; footprint Capacitor_SMD:C_0603_1608Metric -> Capacitor_SMD:C_1206_3216Metric; moved to B.Cu
- C33: value 0.1u -> 20p
- C38: footprint Capacitor_SMD:C_1206_3216Metric -> Capacitor_SMD:C_0603_1608Metric; moved to F.Cu
- C39: value 100n -> 10u; footprint Capacitor_SMD:C_0603_1608Metric -> Capacitor_SMD:C_1206_3216Metric; moved to B.Cu
- C40, C41: value 20p -> 100n
- C44: value 1u -> 270p; moved to B.Cu
- C45: value 4.7u -> 100n; moved to B.Cu
- C46, C48: value 100n -> 27u; footprint Capacitor_SMD:C_0603_1608Metric -> Capacitor_SMD:C_1206_3216Metric; moved to B.Cu
- C47: value 100n -> 22u; footprint Capacitor_SMD:C_0603_1608Metric -> Capacitor_SMD:C_1206_3216Metric; moved to B.Cu
- C5: value 10p -> 100n; moved to B.Cu
- C6: value 0.1u -> 10p; moved to F.Cu
- C8: moved to F.Cu
- C9: value 1n -> 47u; footprint Capacitor_SMD:C_0603_1608Metric -> Capacitor_SMD:CP_Elec_5x5.4
- J2: value connection_moteur -> Conn_01x02_Pin; footprint Connector_JST:JST_EH_B4B-EH-A_1x04_P2.50mm_Vertical -> Connector_JST:JST_EH_B2B-EH-A_1x02_P2.50mm_Vertical
- J3: value Conn_01x05_Pin -> connection_moteur; footprint Connector_PinHeader_1.27mm:PinHeader_1x05_P1.27mm_Vertical -> Connector_JST:JST_EH_B4B-EH-A_1x04_P2.50mm_Vertical
- J4: value Conn_01x03_Pin -> Conn_01x05_Pin; footprint Connector_PinHeader_1.27mm:PinHeader_1x03_P1.27mm_Vertical -> Connector_PinHeader_1.27mm:PinHeader_1x05_P1.27mm_Vertical
- J5: value Conn_01x02_Pin -> Conn_01x03_Pin; footprint Connector_JST:JST_EH_B2B-EH-A_1x02_P2.50mm_Vertical -> Connector_JST:JST_EH_B3B-EH-A_1x03_P2.50mm_Vertical; moved to F.Cu
- R1: value 49.9 -> 47k; moved to B.Cu
- R16: value 12.1k -> 12k
- R2: value 47k -> 49.9; moved to F.Cu
- S1: value TS40-66-43-BK-260-SMT-TR -> B3U-1100PM; footprint footprints:TS40-66-43-BK-260-SMT-TR -> footprints:B3U1100PM
- U1: value HX1188NL -> SP3485CN; footprint footprints:HX1188NL -> Package_SO:SOIC-8_3.9x4.9mm_P1.27mm; moved to B.Cu
- U2: value SP3485CN -> HX1188NL; footprint Package_SO:SOIC-8_3.9x4.9mm_P1.27mm -> footprints:HX1188NL; moved to F.Cu
- moved Q1 100.9 mm to (132.5, 105.4), turned to -90 degrees
- moved R14 98.1 mm to (132.5, 100.8), turned to 180 degrees
- moved R13 98.1 mm to (132.5, 102.3), turned to 0 degrees
- moved J5 98.0 mm to (134.8, 116.2), turned to 0 degrees
- moved C38 92.0 mm to (149.5, 102.5), turned to 180 degrees
- moved D1 91.7 mm to (138.1, 110.9), turned to 180 degrees
- moved R3 90.5 mm to (137.4, 96.5), turned to 180 degrees
- moved R10 86.6 mm to (148.0, 97.0), turned to 90 degrees
- moved R9 86.4 mm to (148.5, 99.7), turned to 180 degrees
- moved R8 85.8 mm to (146.0, 93.5), turned to 180 degrees
- moved D3 81.8 mm to (149.3, 110.9), turned to 180 degrees
- moved L1 79.1 mm to (162.1, 111.5), turned to -90 degrees
- moved J2 79.0 mm to (177.3, 116.2), turned to 0 degrees
- moved C18 74.7 mm to (165.6, 106.2), turned to 90 degrees
- moved R24 66.3 mm to (171.6, 93.8), turned to 90 degrees
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Connections:
- net Net-(IC1-RBIAS) renamed /RBIAS
- net Net-(IC1-VDD33BIAS) renamed /VDD33BIAS
- net Net-(Q1-G) renamed /GATE
- net Net-(U3-A0) renamed /AX
- net Net-(U4-PGOOD) renamed /PGOOD
- net Net-(U4-RT_SYNC) renamed /RT_SYNC
- net Net-(U5-BOOT0) renamed /BOOT0
- net Net-(U5-PA5) renamed /PA5
- net Net-(U5-PA6) renamed /PA6
- net Net-(U5-PA7) renamed /PA7
- C10 pad 1: +12V -> /CMT
- C18 pad 1: Net-(D2-K) -> /VDD33TXRX1
- C19 pad 1: /VDD33TXRX1 -> /VDD33TXRX2
- C20 pad 1: /VDD33TXRX2 -> /VDDCR
- C21 pad 1: /VDDCR -> +3.3V
- C22 pad 1: +3.3V -> GND
- C22 pad 2: GND -> Net-(C22-Pad2)
- C26 pad 1: GND -> /VIN
- C26 pad 2: Net-(C26-Pad2) -> GND
- C27 pad 1: GND -> /VDD12TX1
- C27 pad 2: /OSCO -> GND
- C28 pad 1: +3.3V -> /VDD12TX1
- C29 pad 1: Net-(D2-K) -> /VIN
- C30 pad 1: GND -> /VIN
- C30 pad 2: +3.3V -> GND
- C33 pad 1: /VDD12TX1 -> GND
- C33 pad 2: GND -> /PH1
- C35 pad 1: /VDD12TX1 -> GND
- C35 pad 2: GND -> /NRST
- C38 pad 1: Net-(D2-K) -> +3.3V
- C38 pad 2: GND -> /VDD19
- C39 pad 1: /AVDD -> +12V
- C40 pad 1: GND -> +3.3V
- C40 pad 2: Net-(U5-PH0) -> /VDD32
- C41 pad 1: GND -> +3.3V
- C41 pad 2: Net-(U5-PH1) -> /VDD48
- C42 pad 1: Net-(U4-SS) -> /BOOT
- C42 pad 2: GND -> Net-(D3-K)
- C43 pad 1: GND -> +3.3V
- C43 pad 2: /NRST -> /VDD64
- C44 pad 1: GND -> +12V
- C44 pad 2: +3.3V -> /FB
- C45 pad 1: Net-(U5-VCAP_1) -> /SW
- C45 pad 2: GND -> /BST
- C46 pad 1: +3.3V -> +12V
- C46 pad 2: Net-(C46-Pad2) -> GND
- C47 pad 2: Net-(C47-Pad2) -> GND
- C48 pad 1: +3.3V -> +12V
- C48 pad 2: Net-(C48-Pad2) -> GND
- C5 pad 1: /RXA_N -> +3.3V
- C6 pad 1: +3.3V -> /RXA_N
- C7 pad 1: Net-(U1-RCT) -> /TCT
- C9 pad 1: Net-(C9-Pad1) -> +12V
- D1 pad 1: Net-(D1-K) -> +12V
- D1 pad 2: +12V -> /DRAIN
- D2 pad 1: Net-(D2-K) -> /VIN
- D2 pad 2: +36V -> Net-(D2-A)
- J1 pad 1: Net-(J1-Pin_1) -> /RX_N
- J1 pad 2: Net-(J1-Pin_2) -> /RX_P
- J1 pad 3: Net-(J1-Pin_3) -> /TX_N
- J1 pad 4: Net-(J1-Pin_4) -> /TX_P
- J2 pad 1: Net-(D1-K) -> GND
- J2 pad 2: +12V -> +36V
- J3 pad 1: /SWDIO -> /DRAIN
- J3 pad 2: /SWCLK -> +12V
- J3 pad 3: GND -> /DATA+
- J3 pad 4: +3.3V -> /DATA-
- J4 pad 1: Net-(J4-Pin_1) -> /SWDIO
- J4 pad 2: Net-(J4-Pin_2) -> /SWCLK
- J4 pad 3: Net-(J4-Pin_3) -> GND
- J5 pad 1: GND -> /PA1
- J5 pad 2: +36V -> /PA0
- Q1 pad 3: Net-(D1-K) -> /DRAIN
- R1 pad 1: /VDD33TXRX1 -> GND
- R1 pad 2: /TXA_P -> /RS485_MODE
- R10 pad 1: Net-(J2-Pin_4) -> /DATA-
- R10 pad 2: Net-(J2-Pin_3) -> /DATA+
- R11 pad 1: Net-(C9-Pad1) -> /CMT
- R11 pad 2: Net-(R11-Pad2) -> /CMT1
- R12 pad 1: Net-(C9-Pad1) -> /CMT
- R12 pad 2: Net-(R12-Pad2) -> /CMT2
- R2 pad 1: GND -> /VDD33TXRX1
- R2 pad 2: /RS485_MODE -> /TXA_P
- R20 pad 2: Net-(C26-Pad2) -> Net-(C22-Pad2)
- R23 pad 1: Net-(D2-K) -> /VIN
- R28 pad 2: Net-(U4-FB) -> /FB
- R29 pad 1: Net-(U4-FB) -> /FB
- R3 pad 1: Net-(U2-DE) -> /DE/RE
- R7 pad 2: Net-(U1-RCT) -> /TCT
- R8 pad 1: Net-(J2-Pin_3) -> /DATA+
- R9 pad 2: Net-(J2-Pin_4) -> /DATA-
- S1 pad 1: GND -> /NRST
- S1 pad 3: /NRST -> GND
- U1 pad 1: /TXA_P -> /RO
- U1 pad 2: Net-(U1-RCT) -> /DE/RE
- U1 pad 3: /TXA_N -> /DE/RE
- U1 pad 4: unconnected-(U1-NC-Pad4) -> /DI
- U1 pad 5: unconnected-(U1-NC-Pad5) -> GND
- U1 pad 6: /RXA_P -> /DATA+
- U1 pad 7: Net-(U1-RCT) -> /DATA-
- U1 pad 8: /RXA_N -> +3.3V
- U2 pad 1: /RO -> /TXA_P
- U2 pad 2: Net-(U2-DE) -> /TCT
- U2 pad 3: Net-(U2-DE) -> /TXA_N
- U2 pad 4: /DI -> unconnected-(U2-NC-Pad4)
- U2 pad 5: GND -> unconnected-(U2-NC-Pad5)
- U2 pad 6: Net-(J2-Pin_3) -> /RXA_P
- U2 pad 7: Net-(J2-Pin_4) -> /TCT
- U2 pad 8: +3.3V -> /RXA_N
- U4 pad 1: Net-(U4-BOOT) -> /BOOT
- U4 pad 2: Net-(D2-K) -> /VIN
- U4 pad 3: Net-(D2-K) -> /VIN
- U4 pad 4: Net-(D2-K) -> /VIN
- U4 pad 6: Net-(U4-SS) -> /SS
- U4 pad 7: Net-(U4-FB) -> /FB
- U5 pad 14: Net-(J4-Pin_2) -> /PA0
- U5 pad 15: Net-(J4-Pin_3) -> /PA1
- U5 pad 19: Net-(C46-Pad2) -> /VDD19
- U5 pad 20: Net-(J4-Pin_1) -> /PA4
- U5 pad 30: Net-(U5-VCAP_1) -> /VCAP_1
- U5 pad 32: Net-(C47-Pad2) -> /VDD32
- U5 pad 48: Net-(C48-Pad2) -> /VDD48
- U5 pad 5: Net-(U5-PH0) -> /PH0
- U5 pad 6: Net-(U5-PH1) -> /PH1
- U5 pad 64: Net-(C51-Pad2) -> /VDD64
- Y1 pad 2: Net-(C26-Pad2) -> Net-(C22-Pad2)
- Y2 pad 1: Net-(U5-PH1) -> /PH1
- Y2 pad 2: Net-(U5-PH0) -> /PH0
Routing:
- net GND: track 0.00 -> 132.1 mm, vias 0 -> 78
- net +3.3V: track 0.00 -> 81.0 mm, vias 0 -> 31
- net /DRAIN: track 0.00 -> 80.6 mm
- net /DATA+: track 0.00 -> 72.4 mm
- net /DATA-: track 0.00 -> 58.0 mm
- net +12V: track 18.4 -> 60.0 mm, vias 0 -> 7
- net /RST#: track 0.00 -> 37.7 mm, vias 0 -> 2
- net /SCS#: track 0.00 -> 36.7 mm, vias 0 -> 2
- net /IRQ: track 0.00 -> 30.1 mm, vias 0 -> 2
- net /RXA_N: track 45.2 -> 15.5 mm, vias 0 -> 2
- net /PA0: track 0.00 -> 26.1 mm
- net /PA1: track 0.00 -> 26.0 mm
- net /PA4: track 0.00 -> 24.5 mm
- net /TX_N: track 0.00 -> 24.4 mm
- net /SYNC0: track 0.00 -> 23.4 mm, vias 0 -> 2
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- added copper zone on B.Cu, net +12V
- added copper zone on In2.Cu, net +12V
- added copper zone on B.Cu, net +3.3V
- added copper zone on F.Cu, net +3.3V
- added copper zone on In2.Cu, net +3.3V
- added copper zone on B.Cu, net /GATE
- added copper zone on F.Cu, net /VDDCR
- added copper zone on B.Cu, net GND
- added copper zone on F.Cu, net GND
- added copper zone on In1.Cu, net GND
- added copper zone on In2.Cu, net GND
Other:
- board outline added: 67 x 43 mm
- board text added: "+3.3V"
- board text added: "+36V|GND"
- board text added: "ECAT"
- board text added: "GND"
- board text added: "GND|12V|D+|D-"
- board text added: "GPIO PINS"
- board text added: "Heemskerk Innovative Technology Robot Gripper Controller"
- board text added: "NRST"
- board text added: "PA0"
- board text added: "PA1"
- board text added: "PA4"
- board text added: "PWR"
- board text added: "RS485"
- board text added: "RX_N|RX_P|TX_N|TX_P"
- board text added: "SWCLK"
- board text added: "SWDIO"
- board text removed: "Module RS485"
- board text removed: "Zone EtherCAT (LAN9252)"
- board text removed: "Zone MCU"
- board text removed: "Zone d'alimentation"
- board text removed: "Zone entrée robot"

Commit message: 1KHz ecat communication frequency done
Parts:
- added D4: LED_Small, LED_SMD:LED_0201_0603Metric, F.Cu at (176.3, 80.6)
- added D5: LED_Small, LED_SMD:LED_0201_0603Metric, F.Cu at (174.8, 80.6)
- added R34: 1k, Resistor_SMD:R_0603_1608Metric, F.Cu at (174.7, 83.0)
- added R35: 3.3k, Resistor_SMD:R_0603_1608Metric, F.Cu at (176.3, 83.0)
- moved C6 0.21 mm to (171.0, 106.4)
- moved C7 0.20 mm to (168.8, 106.1)
- moved C35 0.15 mm to (143.2, 87.4)
- moved R31 0.15 mm to (162.3, 106.1)
- moved R15 0.14 mm to (159.6, 111.8)
- moved C18 0.10 mm to (165.7, 106.1)
- moved R16 0.10 mm to (165.9, 95.5)
- moved R12 0.10 mm to (179.6, 100.1)
- moved FB3 0.09 mm to (164.1, 106.1)
- moved FB1 0.08 mm to (165.4, 91.6)
- moved R18 0.08 mm to (165.8, 111.8)
- moved C2 0.06 mm to (171.8, 89.5)
- moved C28 0.06 mm to (162.7, 95.5)
- moved R32 0.06 mm to (144.7, 90.4)
- moved C1 0.06 mm to (152.6, 90.1)
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Routing:
- net +3.3V: track 81.0 -> 89.7 mm
- net +12V: track 60.0 -> 62.4 mm
- net GND: track 132.1 -> 134.2 mm, vias 78 -> 77
- net Net-(D5-A): track 0.00 -> 1.25 mm
- net Net-(D4-A): track 0.00 -> 1.25 mm
